Commit message: finished adding arm / wrist to left hand

File: URDF/ability_hand_left_large-wrist.urdf (robot description, URDF)
Before this commit: robot ability_hand, 19 links, 18 joints
Links:
- added link upper_arm; visual cylinder length=0.34 radius=0.03
- link base: mass 0.200 -> None
- link index_L1: mass 0.00635888 -> None
- link index_L2: mass 0.00645 -> None
- link lower_arm: mass 0.500 -> None; geometry visual cylinder length=0.34 radius=0.03
- link middle_L1: mass 0.00635888 -> None
- link middle_L2: mass 0.00645 -> None
- link pinky_L1: mass 0.00635888 -> None
- link pinky_L2: mass 0.00645 -> None
- link ring_L1: mass 0.00635888 -> None
- link ring_L2: mass 0.00645 -> None
- link thumb_L1: mass 0.00268342 -> None
- link thumb_L2: mass 0.0055 -> None
- link thumb_base: mass 0.400 -> None
- link wrist_link: mass 0.1 -> None; geometry visual box size=0.05 0.02 0.02
Joints:
- added joint elbow: type revolute, parent lower_arm, child upper_arm, origin xyz=0 0 -0.16 rpy=0 0 0, axis 0 1 0, limit lower=-1.57 upper=1.57
- joint idx_anchor: origin xyz=31.5541e-3  -10.44e-3 0.14e-3 rpy=0 0 0 -> xyz=31.5541e-3 -10.44e-3 0.14e-3 rpy=0 0 0
- joint index_q1: limit lower=0 upper=2.0943951 effort=6.0 velocity=8.0677777442 -> lower=0 upper=2.0943951
- joint index_q2: limit lower=0.0 upper=2.6586 effort=6.0 velocity=8.0677777442 -> lower=0.0 upper=2.6586
- joint mid_anchor: origin xyz=31.5541e-3  -10.44e-3 0.14e-3 rpy=0 0 0 -> xyz=31.5541e-3 -10.44e-3 0.14e-3 rpy=0 0 0
- joint middle_q1: limit lower=0 upper=2.0943951 effort=6.0 velocity=8.0677777442 -> lower=0 upper=2.0943951
- joint middle_q2: limit lower=0.0 upper=2.6586 effort=6.0 velocity=8.0677777442 -> lower=0.0 upper=2.6586
- joint pinky_q1: limit lower=0 upper=2.0943951 effort=6.0 velocity=8.0677777442 -> lower=0 upper=2.0943951
- joint pinky_q2: limit lower=0.0 upper=2.6586 effort=6.0 velocity=8.0677777442 -> lower=0.0 upper=2.6586
- joint pnky_anchor: origin xyz=31.5541e-3  -10.44e-3 0.14e-3 rpy=0 0 0 -> xyz=31.5541e-3 -10.44e-3 0.14e-3 rpy=0 0 0
- joint ring_q1: limit lower=0 upper=2.0943951 effort=6.0 velocity=8.0677777442 -> lower=0 upper=2.0943951
- joint ring_q2: limit lower=0.0 upper=2.6586 effort=6.0 velocity=8.0677777442 -> lower=0.0 upper=2.6586
- joint rng_anchor: origin xyz=31.5541e-3  -10.44e-3 0.14e-3 rpy=0 0 0 -> xyz=31.5541e-3 -10.44e-3 0.14e-3 rpy=0 0 0
- joint thmb_anchor: origin xyz=52.0012259e-3  28.0086971e-3 -.884835778e-3 rpy=0 0 0 -> xyz=52.0012259e-3 28.0086971e-3 -.884835778e-3 rpy=0 0 0
- joint thumb_q1: limit lower=-2.0943951 upper=0 effort=1.2 velocity=40.338888721 -> lower=-2.0943951 upper=0
- joint thumb_q2: limit lower=0 upper=2.0943951 effort=6.0 velocity=8.0677777442 -> lower=0 upper=2.0943951
- joint wrist_flexion: limit lower=-1.57 upper=1.57 effort=10.0 velocity=1.0 -> lower=-1.57 upper=1.57; origin xyz=0 0 0.05 rpy=0 0 0 -> xyz=0 0 0.02 rpy=0 0 0
- joint wrist_rotation: limit lower=-3.14 upper=3.14 effort=10.0 velocity=1.0 -> lower=-1.57 upper=1.57; origin xyz=0 0 0.15 rpy=0 0 0 -> xyz=0 0 0.0 rpy=0 0 0

Commit message: added urdf for right hand / arm

File: URDF/ability_hand_left_large-wrist.urdf (robot description, URDF)
Before this commit: robot ability_hand, 20 links, 19 joints
Joints:
- joint wrist_rotation: limit lower=-1.57 upper=1.57 -> lower=-3.14 upper=3.14

File: URDF/ability_hand_right_large.urdf (robot description, URDF)
Before this commit: robot ability_hand, 17 links, 16 joints
Links:
- link index_L2: geometry visual mesh filename=models/idx-F2-Lg.STL
